File: pcb/egret.kicad_pcb (KiCad board)
At the start: 2 copper layers, 223.1 x 94.9 mm, 100 parts

Commit message: v1.0 pcb design, gitignore
Other:
- board text added: "egret v1.0 by rschenk"
Changed lines of the file:
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@@
     )
     (pad_to_mask_clearance 0.05)
+    (grid_origin 197.975 120.075)
     (pcbplotparams
       (layerselection 0x00010fc_ffffffff)
@@
       (outputformat 1)
       (mirror false)
-      (drillshape 1)
+      (drillshape 0)
       (scaleselection 1)
-      (outputdirectory "")
+      (outputdirectory "../gerbers/")
     )
   )
@@
   (gr_line (start 162.45063 70.905944) (end 177.841225 73.619501) (layer "Edge.Cuts") (width 0.151694))
   (gr_line (start 141.107414 64.876372) (end 141.162383 64.859446) (layer "Edge.Cuts") (width 0.151694))
-  (gr_text "face up" (at 207.725 99.5 90) (layer "F.SilkS")
+  (gr_text "egret v1.0 by rschenk" (at 207.725 99.5 90) (layer "F.SilkS")
+    (effects (font (size 1 1) (thickness 0.15)))
+  )
+  (gr_text "face up" (at 206.425 83.5) (layer "F.SilkS")
     (effects (font (size 1 1) (thickness 0.15)))
   )
